File: PCB/pcb/pcb.kicad_sch (KiCad schematic)
At the start: 5 parts, among them U1 XT60PW-F, U2 XT60PW-M, U3 LM78L05ACM, U4 BTS2140

Commit message: add
Parts:
- added J1: 09662527611, Library:09662527611, symbol simple_ae:09662527611
- added U5: HC-06, Library:HC-06, symbol simple_ae:HC-06
- added U6: Switch_4_Voies, Library:DIP-8_300_ELL, symbol simple_ae:Switch_4_Voies
Connections:
- net +12V: now also U1.1, J1.7, J1.8; no longer U1.2
- net +5V: now also J1.1, J1.2, U5.5 (VCC)
- net GND: now also J1.3, J1.4, J1.MH1, J1.MH2, U5.4 (GND)
- net at U4.2 (Collector): now also U1.2; no longer U1.1
- net TXD_2: now reaches XA1.D0 (D0_RX0)
- net TXD_2: now also U6.5, U6.8
- net RXD_2: now reaches XA1.D1 (D1_TX0)
- net RXD_2: now also U6.6, U6.7
- net Cible: now reaches XA1.D2 (D2_INT0)
- net Cible: now also J1.10, J1.11, J1.12, J1.9
- net D4 renamed Bob
- new net RXD: U5.2 (RXD), U6.2, U6.4
- new net TXD: U5.3 (TXD), U6.1, U6.3
Other:
- moved on the sheet: U1
