File: PCB/pcb/pcb.kicad_pcb (KiCad board)
At the start: 2 copper layers, 5 parts, among them U1 XT60PW-F, U2 XT60PW-M, U3 LM78L05ACM, U4 BTS2140

Commit message: add
Parts:
- added J1: 09662527611, Library:09662527611, F.Cu at (146.4, 80.7)
- added U5: HC-06, Library:HC-06, F.Cu at (157.5, 88.9)
- added U6: Switch_4_Voies, Library:DIP-8_300_ELL, F.Cu at (212.1, 54.6)
- moved U2 172.2 mm to (231.2, 59.7), turned to -90 degrees
- moved U1 154.3 mm to (231.2, 82.5), turned to -90 degrees
- moved U4 75.4 mm to (212.1, 83.9), turned to -90 degrees
- moved U3 66.1 mm to (212.1, 64.8)
- moved XA1 61.8 mm to (188.0, 91.9)
Connections:
- U1 pad 1: unconnected-(U1-Pad1) -> +12V
- U1 pad 2: unconnected-(U1-Pad2) -> Net-(U1-Pad2)
- U2 pad 1: unconnected-(U2-Pad1) -> GND
- U2 pad 2: unconnected-(U2-Pad2) -> +12V
- U3 pad 1: unconnected-(U3-Pad1) -> +5V
- U3 pad 2: Net-(U3-Pad2) -> GND
- U3 pad 3: Net-(U3-Pad2) -> GND
- U3 pad 6: Net-(U3-Pad2) -> GND
- U3 pad 7: Net-(U3-Pad2) -> GND
- U3 pad 8: unconnected-(U3-Pad8) -> +12V
- U4 pad 1: unconnected-(U4-Pad1) -> Bob
- U4 pad 2: unconnected-(U4-Pad2) -> Net-(U1-Pad2)
- U4 pad 3: unconnected-(U4-Pad3) -> GND
- XA1 pad 5V: unconnected-(XA1-Pad5V) -> +5V
- XA1 pad D0: unconnected-(XA1-PadD0) -> TXD_2
- XA1 pad D1: unconnected-(XA1-PadD1) -> RXD_2
- XA1 pad D2: unconnected-(XA1-PadD2) -> Cible
- XA1 pad D4: unconnected-(XA1-PadD4) -> Bob
- XA1 pad GND1: unconnected-(XA1-PadGND1) -> GND
- XA1 pad GND2: unconnected-(XA1-PadGND2) -> GND
Routing:
- net +12V: track 0.00 -> 132.4 mm, vias 0 -> 1
- net RXD: track 0.00 -> 100.0 mm
- net TXD: track 0.00 -> 93.5 mm
- net Bob: track 0.00 -> 87.4 mm, vias 0 -> 2
- net Cible: track 0.00 -> 56.6 mm
- net TXD_2: track 0.00 -> 45.4 mm
- net GND: track 0.00 -> 40.7 mm
- net RXD_2: track 0.00 -> 38.8 mm
- net Net-(U1-Pad2): track 0.00 -> 19.7 mm
- net +5V: track 0.00 -> 15.1 mm
- added copper zone on B.Cu, net +5V
- added copper zone on F.Cu, net GND
Other:
- board outline added: 101.6 x 51.7 mm

Commit message: ddd
Parts:
- moved XA1 43.5 mm to (194.9, 49.0), turned to 180 degrees
- moved J1 11.4 mm to (157.9, 80.7)
- moved U5 8.89 mm to (166.4, 88.9)
Routing:
- net Cible: track 56.6 -> 84.2 mm, vias 0 -> 2
- net Bob: track 87.4 -> 70.0 mm
- net +5V: track 15.1 -> 1.93 mm, vias 0 -> 1
- net RXD: track 100.0 -> 87.8 mm
- net TXD: track 93.5 -> 82.1 mm
- net +12V: track 132.4 -> 121.0 mm
- net TXD_2: track 45.4 -> 52.7 mm
- net RXD_2: track 38.8 -> 45.7 mm
Other:
- board size 101.6 x 51.7 mm -> 87.6 x 57.1 mm
